File: Ruler/Ruler.kicad_sch (KiCad schematic)
At the start: 2 parts

Commit message: 表面完成
Parts:
- added D1: ~, Diode_SMD:D_SOD-123, symbol Diode:1N4148WT
- added D2: ~, Diode_SMD:D_SOD-323, symbol Diode:1N4148WT
- added D3: ~, Diode_SMD:D_SMA, symbol Diode:1N4148WT
- added D4: ~, Diode_SMD:D_SMB, symbol Diode:1N4148WT
- added Q1: NPN, Package_TO_SOT_SMD:SOT-23, symbol Simulation_SPICE:NPN
- added Q2: NPN, Package_TO_SOT_SMD:SOT-223, symbol Simulation_SPICE:NPN
- added Q3: NPN, Package_TO_SOT_SMD:SOT-89-3, symbol Simulation_SPICE:NPN
- added Q4: NPN, Package_TO_SOT_SMD:TO-252-2, symbol Simulation_SPICE:NPN
- added R3: R, Resistor_SMD:R_0603_1608Metric, symbol Device:R
- added R4: R, Resistor_SMD:R_0805_2012Metric, symbol Device:R
- added R5: R, Resistor_SMD:R_1206_3216Metric, symbol Device:R
- added R6: R, Resistor_SMD:R_1210_3225Metric, symbol Device:R
- added TP1: TestPoint, TestPoint:TestPoint_Pad_D1.0mm, symbol Connector:TestPoint
- added TP2: TestPoint, TestPoint:TestPoint_Pad_D1.5mm, symbol Connector:TestPoint
- added TP3: TestPoint, TestPoint:TestPoint_Pad_D2.0mm, symbol Connector:TestPoint
- added TP4: TestPoint, TestPoint:TestPoint_Pad_D2.5mm, symbol Connector:TestPoint
- added U1: IR2302, Package_SO:SOIC-8_3.9x4.9mm_P1.27mm, symbol Driver_FET:IR2302
- added U3: STM32F303K8Tx, Package_QFP:LQFP-32_7x7mm_P0.8mm, symbol MCU_ST_STM32F3:STM32F303K8Tx
- R2: footprint Resistor_SMD:R_0201_0603Metric -> Resistor_SMD:R_0402_1005Metric
Connections:
- new net: U3.16 (VSS), U3.32 (VSS)

Commit message: 裏面途中
Parts:
- added H1: MountingHole, MountingHole:MountingHole_2.2mm_M2_Pad_Via, symbol Mechanical:MountingHole
- renumbered U3 to U2
Changed lines of the file:
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@@
 		(dnp no)
 		(fields_autoplaced yes)
-		(property "Reference" "U3"
+		(property "Reference" "U2"
 			(at 38.9733 168.91 0)
 			(effects
@@
 			(project ""
 				(path "/31eb4b57-0a31-442e-bed8-5e9cc9d6f7cf"
-					(reference "U3")
+					(reference "U2")
 					(unit 1)
 				)
@@
 					(unit 1)
 				)
+			)
+		)
+	)
+	(symbol
+		(lib_id "Mechanical:MountingHole")
+		(at 41.91 82.55 0)
+		(unit 1)
+		(exclude_from_sim no)
+		(in_bom no)
+		(on_board yes)
+		(dnp no)
+		(fields_autoplaced yes)
+		(property "Reference" "H1"
+			(at 44.45 81.2799 0)
+			(effects
+				(font
+					(size 1.27 1.27)
+				)
+				(justify left)
+			)
+		)
+		(property "Value" "MountingHole"
+			(at 44.45 83.8199 0)
+			(effects
+				(font
+					(size 1.27 1.27)
+				)
+				(justify left)
+			)
+		)
+		(property "Footprint" "MountingHole:MountingHole_2.2mm_M2_Pad_Via"
+			(at 41.91 82.55 0)
+			(effects
+				(font
+					(size 1.27 1.27)
+				)
+				(hide yes)
+			)
+		)
+		(property "Datasheet" "~"
+			(at 41.91 82.55 0)
+			(effects
+				(font
+					(size 1.27 1.27)
+				)
+				(hide yes)
+			)
+		)
+		(property "Description" "Mounting Hole without connection"
+			(at 41.91 82.55 0)
+			(effects
+				(font
+					(size 1.27 1.27)
+				)
+				(hide yes)
+			)
+		)
+		(instances
+			(project ""
+				(path "/31eb4b57-0a31-442e-bed8-5e9cc9d6f7cf"
+					(reference "H1")
+					(unit 1)
+				)
