File: Ruler/Ruler.kicad_pcb (KiCad board)
At the start: 2 copper layers, 100 x 25 mm, 0 parts

Commit message: 表面完成
Parts:
- added D1: ~, Diode_SMD:D_SOD-123, F.Cu at (173.8, 111.0)
- added D2: ~, Diode_SMD:D_SOD-323, F.Cu at (173.8, 106.8)
- added D3: ~, Diode_SMD:D_SMA, F.Cu at (173.8, 116.0)
- added D4: ~, Diode_SMD:D_SMB, F.Cu at (182.0, 115.5)
- added Q1: NPN, Package_TO_SOT_SMD:SOT-23, F.Cu at (153.2, 115.2)
- added Q2: NPN, Package_TO_SOT_SMD:SOT-223, F.Cu at (161.2, 116.0)
- added Q3: NPN, Package_TO_SOT_SMD:SOT-89-3, F.Cu at (153.2, 108.2)
- added Q4: NPN, Package_TO_SOT_SMD:TO-252-2, F.Cu at (161.4, 108.7)
- added R1: R, Resistor_SMD:R_0201_0603Metric, F.Cu at (142.2, 106.8)
- added R2: R, Resistor_SMD:R_0402_1005Metric, F.Cu at (142.2, 108.2)
- added R3: R, Resistor_SMD:R_0603_1608Metric, F.Cu at (142.2, 109.8)
- added R4: R, Resistor_SMD:R_0805_2012Metric, F.Cu at (142.2, 111.8)
- added R5: R, Resistor_SMD:R_1206_3216Metric, F.Cu at (142.2, 114.2)
- added R6: R, Resistor_SMD:R_1210_3225Metric, F.Cu at (142.2, 117.2)
- added TP1: TestPoint, TestPoint:TestPoint_Pad_D1.0mm, F.Cu at (135.2, 117.2)
- added TP2: TestPoint, TestPoint:TestPoint_Pad_D1.5mm, F.Cu at (135.2, 115.0)
- added TP3: TestPoint, TestPoint:TestPoint_Pad_D2.0mm, F.Cu at (135.2, 112.2)
- added TP4: TestPoint, TestPoint:TestPoint_Pad_D2.5mm, F.Cu at (135.2, 108.8)
- added U1: IR2302, Package_SO:SOIC-8_3.9x4.9mm_P1.27mm, F.Cu at (181.8, 109.0)
- added U3: STM32F303K8Tx, Package_QFP:LQFP-32_7x7mm_P0.8mm, F.Cu at (193.2, 111.8)
Other:
- board text added: "0.2"
- board text added: "0.3"
- board text added: "0.5"
- board text added: "0.75"
- board text added: "0603"
- board text added: "1.0"
- board text added: "1.0mm"
- board text added: "1.5"
- board text added: "1.5mm"
- board text added: "1005"
- board text added: "1608"
- board text added: "2.0mm"
- board text added: "2.5mm"
- board text added: "2012"
- board text added: "3216"
- board text added: "3225"
- board text added: "LQFP32"
- board text added: "SMA"
- board text added: "SMB"
- board text added: "SOD123"
- board text added: "SOD323"
- board text added: "SOIC8"
- board text added: "SOT223"
- board text added: "SOT23"
- board text added: "SOT89"
- board text added: "Silk"
- board text added: "TO252"
- board text added: "Trace"
- board text added: "mm"

Commit message: 裏面途中
Parts:
- removed U3: STM32F303K8Tx, Package_QFP:LQFP-32_7x7mm_P0.8mm
- added H1: MountingHole, MountingHole:MountingHole_2.2mm_M2_Pad_Via, F.Cu at (102.2, 102.2)
- added U2: STM32F303K8Tx, Package_QFP:LQFP-32_7x7mm_P0.8mm, F.Cu at (191.5, 111.8)
- moved D1 1.75 mm to (172.0, 111.0)
- moved D2 1.75 mm to (172.1, 106.8)
- moved D3 1.75 mm to (172.0, 116.0)
- moved D4 1.75 mm to (180.2, 115.5)
- moved Q1 1.75 mm to (151.5, 115.2)
- moved Q2 1.75 mm to (159.5, 116.0)
- moved Q3 1.75 mm to (151.5, 108.2)
- moved Q4 1.75 mm to (159.7, 108.7)
- moved R1 1.75 mm to (140.5, 106.8)
- moved R2 1.75 mm to (140.5, 108.2)
- moved R3 1.75 mm to (140.5, 109.8)
- moved R4 1.75 mm to (140.5, 111.8)
- moved R5 1.75 mm to (140.5, 114.2)
- moved R6 1.75 mm to (140.5, 117.2)
- moved U1 1.75 mm to (180.0, 109.0)
Other:
- outline, holes or cut-outs redrawn
- board text added: "B"
- board text added: "C"
- board text added: "D"
- board text added: "Designed by Takumi BAMBA"
- board text added: "Diode"
- board text added: "E"
- board text added: "G"
- board text added: "LED"
- board text added: "MOSFET"
- board text added: "NPN"
- board text added: "Nch"
- board text added: "Normal"
- board text added: "PNP"
- board text added: "Pch"
- board text added: "Photo"
- board text added: "S"
- board text added: "Schottky"
- board text added: "Transistor"
- board text added: "Varactor"

Commit message: 発注した
Parts:
- added G***: LOGO, 0MyLibrary:JLCPCB_40mm, B.Cu at (172.6, 115.5)
- added G***: LOGO, 0MyLibrary:KiCad_20mm, B.Cu at (182.6, 108.2)
- moved TP1 3.75 mm to (139.0, 117.2)
- moved TP2 3.75 mm to (139.0, 115.0)
- moved TP3 3.75 mm to (139.0, 112.2)
- moved TP4 3.75 mm to (139.0, 108.8)
- moved R1 3.54 mm to (144.0, 106.8)
- moved R2 3.54 mm to (144.0, 108.2)
- moved R3 3.54 mm to (144.0, 109.8)
- moved R4 3.54 mm to (144.0, 111.8)
- moved R5 3.54 mm to (144.0, 114.2)
- moved R6 3.54 mm to (144.0, 117.2)
- moved Q1 3.25 mm to (154.8, 115.2)
- moved Q2 3.25 mm to (162.8, 116.0)
- moved Q3 3.25 mm to (154.8, 108.2)
- moved Q4 3.25 mm to (162.9, 108.7)
- moved D1 2.50 mm to (174.5, 111.0)
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Routing:
- net (no net): vias 0 -> 6
Other:
- board text added: "0.4"
- board text added: "0.6"
- board text added: "0.7"
- board text added: "0.8"
- board text added: "Takumi BAMBA"
- board text added: "Via"
- board text removed: "Designed by Takumi BAMBA"
